Commit message: tailsitter dynamics tested

File: rotors_description/urdf/fixed_wing_base.xacro (robot description, xacro)
@@ -123,5 +123,5 @@
     params="robot_namespace suffix parent mass_propeller propeller_radius color
       use_mesh_file mesh_file *origin *inertia">
-    <joint name="${robot_namespace}/propeller_{suffix}_joint" type="continuous">
+    <joint name="${robot_namespace}/propeller_${suffix}_joint" type="continuous">
       <xacro:insert_block name="origin" />
       <axis xyz="0 0 1" />
